File: Hardware/Top/cataclysm-TOP.brd (EAGLE design)
At the start: 38 x 38 mm, 65 parts, among them SW1 SWITCH.MOM, SW2 SWITCH.MOM, U2 NRF52832_MODULE_MDBT42, U4 PCF8523, U5 FT231XS

Commit message: Updated top board
Parts:
- removed C10: 300p, LinnesLab-Passives:C0603
- removed C22: 100n, LinnesLab-Passives:C0603
- removed C23, C24: 47p, LinnesLab-Passives:C0603
- removed C9: (no value), LinnesLab-Passives:C0603
- removed CHRG2: MCP73831, LinnesLab-Power:SOT23-5
- removed CORTEX1: CORTEX_DEBUG_PTH, LinnesLab-Connectors:2X5-PTH-1.27MM
- removed D4, D5: (no value), LinnesLab-DiscreteSemi:USC
- removed JP2: (no value), LinnesLab-Switches:SMT-JUMPER_2_NO_SILK
- removed L2: 10u, LinnesLab-Passives:L0603
- removed LDO2: MIC5504, LinnesLab-Power:SOT23-5
- removed LED5: RED, LinnesLab-LED:LED-0603
- removed LED6: YELLOW, LinnesLab-LED:LED-0603
- removed R19, R20: 1k, LinnesLab-Passives:R0603
- removed R5: 10k, LinnesLab-Passives:R0603
- removed U5: FT231XS, LinnesLab-DigitalIC:SSOP20_L
- removed XTAL3: 32.7680kHz, LinnesLab-Clocks:2-SMD.NOLEAD.2.0MMTO1.2MM
- added C1: 4.7u, LinnesLab-Passives:C0603
- added C3: 1u, LinnesLab-Passives:C0603
- added C4: 10u, LinnesLab-Passives:C0805
- added CHRG1: MCP73831, LinnesLab-Power:SOT23-5
- added D2, D3: (no value), LinnesLab-DiscreteSemi:USC
- added DEBUG1: CORTEX_DEBUG_PTH, LinnesLab-Connectors:2X5-PTH-1.27MM
- added JP1: (no value), LinnesLab-Switches:SMT-JUMPER_2_NO_SILK
- added L1: 10u, LinnesLab-Passives:L0603
- added LDO1: MIC5504, LinnesLab-Power:SOT23-5
- added LED1: RED, LinnesLab-LED:LED-0603
- added LED2: BLUE, LinnesLab-LED:LED-0603
- added R10, R16: 1k, LinnesLab-Passives:R0603
- added U1: NRF52832_MODULE_MDBT42, LinnesLab-Microcontrollers:BLE_MODULE_RAYTAC_MDBT42
- added XTAL1: 32.768kHz, LinnesLab-Clocks:2-SMD.NOLEAD.2.0MMTO1.2MM
- C11: value 300p -> 100n
- C12: value 10u -> 10uF; device LinnesLab-Passives:C0805 -> LinnesLab-Passives:C0603
- C14: value 100n -> 2.2uF; device LinnesLab-Passives:C0603 -> LinnesLab-Passives:C0402
- C16: value 10uF -> 2.2uF; device LinnesLab-Passives:C0603 -> LinnesLab-Passives:C0402
- C18, C19: value 2.2uF -> 47p; device LinnesLab-Passives:C0402 -> LinnesLab-Passives:C0603
- C20: value 4.7u -> 100n
- C21: value 4.7u -> 1u
- C5, C7: value 1u -> (none)
- C8: value (none) -> 4.7u
- J1: device LinnesLab-Connectors:1X07_1.27MM -> LinnesLab-Connectors:1X02
- J2: device LinnesLab-Connectors:1X02 -> LinnesLab-Connectors:1X07_1.27MM
- LED4: value BLUE -> YELLOW
- R1, R2: value 0 -> 10k
- R11: value (none) -> 10k
- R12: value 100k -> 390k
- R13, R14: value 100k -> 27
- R15: value 100k -> 1k
- R17, R18: value 27 -> 0
- R3: value 1k -> 100k
- R4: value 1k -> (none)
- R6: value 10k -> 100k
- R7: value 390k -> 100k
- R9: value 10k -> 1k
- SW1, SW2: value SWITCH.MOM -> (none); device LinnesLab-Switches:TACTILE_SWITCH_SMD_6.2MM_TALL -> LinnesLab-Switches:BUTTON-GULLWING
- SW3, SW4: value (none) -> SWITCH.MOM; device LinnesLab-Switches:BUTTON-GULLWING -> LinnesLab-Switches:TACTILE_SWITCH_SMD_6.2MM_TALL
- U2: value NRF52832_MODULE_MDBT42 -> (none); device LinnesLab-Microcontrollers:BLE_MODULE_RAYTAC_MDBT42 -> LinnesLab-Displays:UG-2864HSWEG01_0.96IN_NO-WRAPAROUND
- U3: value (none) -> FT231XS; device LinnesLab-Displays:UG-2864HSWEG01_0.96IN_NO-WRAPAROUND -> LinnesLab-DigitalIC:SSOP20_L
- XTAL2: value 32.768kHz -> 32.7680kHz
- moved R9 96.6 mm to (41.3, 71.1), turned to 180 degrees
- moved R18 75.0 mm to (5.17, 12.6)
- moved SW2 73.7 mm to (36.2, 77.5)
- moved R8 70.3 mm to (50.6, 30.4), turned to 90 degrees
- moved SW1 68.6 mm to (35.0, 71.4), turned to 180 degrees
- moved R17 65.2 mm to (17.7, 11.2)
- moved XTAL2 48.7 mm to (-18.8, 30.2), turned to 90 degrees
- moved R2 44.9 mm to (9.17, 36.1)
- moved D1 42.2 mm to (8.26, 3.94), flipped to the bottom, turned to 270 degrees
- moved C21 41.2 mm to (-14.5, 25.1), flipped to the top, turned to 180 degrees
- moved R1 41.2 mm to (5.61, 36.1)
- moved SW3 36.8 mm to (22.5, 4.77), turned to 180 degrees
- moved LED4 32.9 mm to (15.8, 9.51), turned to 180 degrees
- moved LED3 32.7 mm to (15.6, 7.39), turned to 180 degrees
- moved R3 30.5 mm to (13.5, 9.01), flipped to the bottom, turned to 270 degrees
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- renumbered SD3 to SD1, USB2 to USB1
Connections:
- removed net A7/TIA: J1.5
- removed net N$24: J1.4
- removed net N$29: J1.3
- removed net N$30: J1.2
- removed net N$31: J1.1
- net !CTS: now also JP1.2, U3.9; no longer JP2.2, U5.9
- net !DTR: now also U3.1; no longer U5.1
- net 3.3V: now also C16.2, C20.2, C21.1, C4.2, D3.-, DEBUG1.1, J2.4, LDO1.5, LED3.A, LED4.A, R1.2, R2.2, U1.11, U2.6, U2.9, U3.14, U3.3; no longer C12.2, C19.2, C2.1, C22.2, CORTEX1.1, D1.-, LDO2.5, LED5.A, LED6.A, R15.2, R5.2, R9.2, U2.11, U3.6, U3.9, U5.14, U5.3
- net A4/BATT: now also R6.1, R7.2, U1.5; no longer U2.5
- net A6/TIA: now also J2.6, U1.7; no longer U2.7
- net A7/PPG: now also J2.7, U1.8; no longer J1.7, U2.8
- net D11/SW1: now also SW3.A1, U1.25; no longer SW1.A1, U2.25
- net D15/SW2: now also SW4.A1, U1.29; no longer SW2.A1, U2.29
- net D16/CS.OLED: now also U1.30, U2.13; no longer U2.30, U3.13
- net D27/CHRG.STATUS: now also CHRG1.1, R3.1, U1.4; no longer CHRG2.1, R12.1, R13.1, R14.2, U2.4
- net D29/LED.CTRL: now also J2.5, U1.6; no longer J1.6, U2.6
- net D3/RESET.OLED: now also U1.17, U2.14; no longer U2.17, U3.14
- net D4/DC.OLED: now also U1.16, U2.15; no longer U2.16, U3.15
- net D7/SD.CS: now also U1.20; no longer U2.20
- net DFU: now also SW2.3, U1.34; no longer SW3.3, U2.34
- net DS/CD1: now also U1.18; no longer U2.18
- net DTR: now also C11.1; no longer C14.1
- net FRST: now also U1.38; no longer U2.38
- net FT3V3: now also U3.13; no longer U5.13
- net GND: now also C1.1, C14.1, C19.2, C20.1, C21.2, C3.1, C4.1, C8.2, CHRG1.2, DEBUG1.3, DEBUG1.5, DEBUG1.7, DEBUG1.9, J1.1, J2.3, JP1.1, LDO1.2, LED1.C, LED2.C, R12.2, R4.1, R7.1, SW1.3, SW2.1, SW3.B1, SW4.B1, U1.1, U1.12, U1.24, U1.39, U2.10, U2.29, U2.30, U2.8, U3.16, U3.6; no longer C10.2, C11.2, C19.1, C20.2, C21.1, C22.1, C23.2, C24.1, C8.1, C9.2, CHRG2.2, CORTEX1.3, CORTEX1.5, CORTEX1.7, CORTEX1.9, J2.1, JP2.1, LDO2.2, LED3.C, LED4.C, R14.1, R15.1, R6.1, R7.2, SW1.B1, SW2.B1, SW3.1, SW4.3, U2.24, U2.39, U3.1, U3.10, U3.12, U3.29, U3.30, U3.8, U5.16, U5.6
- net LED1: now also R9.2, U1.31; no longer R3.2, U2.31
- net LED2: now also R10.2, U1.33; no longer R4.2, U2.33
- net MISO: now also U1.28; no longer U2.28
- net MOSI: now also U1.27, U2.19; no longer U2.27, U3.19
- net N$1: now also R11.2, U2.11; no longer R6.2, U3.11
- net N$10: now also LED2.A, R10.1; no longer LED4.A, R4.1
- net N$11: now also L1.1, U1.10; no longer L2.1, U2.10
- net N$12: now also C2.1, L1.2, U1.9; no longer C7.1, L2.2, U2.9
- net N$13: now also C12.2, U2.28; no longer C16.2, U3.28
- net N$14: now also DEBUG1.8; no longer CORTEX1.8
- net N$15: now also C14.2, U2.27; no longer C18.2, U3.27
- net N$16: now also SW4.B2; no longer SW2.B2
- net N$17: now also CHRG1.5, R4.2; no longer CHRG2.5, R11.2
- net N$19: now also XTAL2.P$1; no longer XTAL3.P$1
- net N$2: now also R12.1, U2.26; no longer R7.1, U3.26
- net N$20: now also XTAL2.P$2; no longer XTAL3.P$2
- net N$21: now also SW3.B2; no longer SW1.B2
- net N$25: now also R13.2, U3.12; no longer R17.2, U5.12
- net N$26: now also R14.2, U3.11; no longer R18.2, U5.11
- net N$27: now also LED3.C, R15.2; no longer LED5.C, R19.2
- net N$28: now also LED4.C, R16.2; no longer LED6.C, R20.2
- net N$3: now also C15.2, U2.2; no longer C13.2, U3.2
- net N$4: now also C5.2, U1.13, XTAL1.P$1; no longer C8.2, U2.13, XTAL2.P$1
- net N$5: now also C15.1, U2.3; no longer C13.1, U3.3
- net N$6: now also C7.1, U1.14, XTAL1.P$2; no longer C9.1, U2.14, XTAL2.P$2
- net N$7: now also C13.2, U2.4; no longer C15.2, U3.4
- net N$8: now also C13.1, U2.5; no longer C15.1, U3.5
- net N$9: now also LED1.A, R9.1; no longer LED3.A, R3.1
- net P0.09/NFC1: now also U1.22; no longer C11.1, U2.22
- net P0.10/NFC2: now also U1.23; no longer C10.1, U2.23
- net RESET: now also C11.2, D3.+, DEBUG1.10, R8.1, SW1.1, U1.35; no longer C14.2, CORTEX1.10, D1.+, R5.1, SW4.1, U2.35
- net RXD.FT: now also R18.1, U3.4; no longer R2.1, U5.4
- net RXD.NRF: now also R17.2, U1.21; no longer R1.2, U2.21
- net RXLED: now also R15.1, U3.17; no longer R19.1, U5.17
- net SCK: now also U1.26, U2.18; no longer U2.26, U3.18
- net SCL: now also J2.2, R2.1, U1.3; no longer R9.1, U2.3
- net SDA: now also J2.1, R1.1, U1.2; no longer R8.1, U2.2
- net SWCLK: now also DEBUG1.4, U1.36; no longer CORTEX1.4, U2.36
- net SWDIO: now also DEBUG1.2, U1.37; no longer CORTEX1.2, U2.37
- net SWO: now also DEBUG1.6, U1.32; no longer CORTEX1.6, U2.32
- net TXD.FT: now also R17.1, U3.20; no longer R1.1, U5.20
- net TXD.NRF: now also R18.2, U1.19; no longer R2.2, U2.19
- net TXLED: now also R16.1, U3.10; no longer R20.1, U5.10
- net USB+: now also C19.1, R14.1; no longer C23.1, R18.1
- net USB-: now also C18.2, R13.1; no longer C24.2, R17.1
- net VIN: now also C1.2, C3.2, CHRG1.4, D1.-, D2.-, LDO1.1, LDO1.3, R3.2; no longer C21.2, C5.2, CHRG2.4, D4.-, D5.-, LDO2.1, LDO2.3, R12.2
- net VLIPO: now also C8.1, CHRG1.3, D1.+, J1.2, R6.2; no longer C20.1, CHRG2.3, D4.+, J2.2, R13.2
- net V_USB: now also D2.+, U3.15; no longer D5.+, U5.15
Routing:
- net GND: track 0.00 -> 28.3 mm, vias 0 -> 19
- net USB-: track 0.00 -> 24.3 mm, vias 0 -> 1
- net VLIPO: track 0.00 -> 22.4 mm
- net USB+: track 0.00 -> 14.9 mm, vias 0 -> 1
- net VIN: track 0.00 -> 12.6 mm
- net TXD.FT: track 0.00 -> 8.21 mm
- net N$3: track 0.00 -> 5.77 mm
- net N$6: track 0.00 -> 5.59 mm
- net N$4: track 0.00 -> 5.33 mm
- net N$7: track 0.00 -> 4.62 mm
- net N$12: track 0.00 -> 4.22 mm
- net N$5: track 0.00 -> 4.21 mm
- net N$8: track 0.00 -> 3.05 mm
- net N$15: track 0.00 -> 2.78 mm
- net N$11: track 0.00 -> 2.38 mm
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- added copper zone on layer 1, net 3.3V
- added copper zone on layer 16, net GND

Commit message: Almost finished with take 8
Parts:
- removed C21: 1u, LinnesLab-Passives:C0603
- removed SD1: (no value), LinnesLab-Connectors:MICROSD
- removed U4: PCF8523, LinnesLab-Clocks:SO8
- removed XTAL1: 32.768kHz, LinnesLab-Clocks:2-SMD.NOLEAD.2.0MMTO1.2MM
- removed XTAL2: 32.7680kHz, LinnesLab-Clocks:2-SMD.NOLEAD.2.0MMTO1.2MM
- added Y1: 32.768kHz, LinnesLab-Clocks:2-SMD.NOLEAD.2.0MMTO1.2MM
- C1: value 4.7u -> 1u
- C14: device LinnesLab-Passives:C0402 -> LinnesLab-Passives:C0603
- C3: value 1u -> 4.7u
- moved LED2 58.8 mm to (34.6, 20.1), turned to 270 degrees
- moved SW1 55.3 mm to (34.6, 16.1)
- moved R10 55.0 mm to (34.6, 23.3), turned to 90 degrees
- moved LED1 51.7 mm to (32.4, 20.3), turned to 270 degrees
- moved R9 48.5 mm to (32.4, 23.4), turned to 90 degrees
- moved SW2 41.9 mm to (34.9, 35.7), turned to 180 degrees
- moved C11 29.3 mm to (35.2, 10.8), turned to 0 degrees
- moved C3 27.7 mm to (3.14, 30.5), flipped to the top
- moved D3 25.3 mm to (34.8, 12.2), turned to 180 degrees
- moved LDO1 24.2 mm to (-2.09, -14.9), flipped to the top, turned to 0 degrees
- moved C6 24.0 mm to (-2.82, -11.1), flipped to the top
- moved R3 23.0 mm to (5.29, 30.5), flipped to the top, turned to 90 degrees
- moved R8 22.8 mm to (34.8, 13.9), turned to 180 degrees
- moved C1 22.3 mm to (4.76, 27.0), flipped to the top, turned to 90 degrees
- moved R4 21.7 mm to (1.35, 30.6), flipped to the top, turned to 270 degrees
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Connections:
- removed net !DTR: U3.1
- removed net A4/BATT: R6.1, R7.2, U1.5
- removed net A7/PPG: J2.7, U1.8
- removed net CD2: SD1.CD2
- removed net N$19: U4.2, XTAL2.P$1
- removed net N$20: U4.1, XTAL2.P$2
- removed net VBAT: U4.3
- new net A4/PPG: J2.7, U1.5
- new net A7/BATT: R6.1, R7.2, U1.8
- new net VIN1: C1.2, C3.2, CHRG1.4, LDO1.1, LDO1.3, R3.2
- net 3.3V: no longer C21.1, SD1.4, U4.8
- net A6/TIA: now also J2.5; no longer J2.6
- net D29/LED.CTRL: now also J2.6; no longer J2.5
- net D7/SD.CS: no longer SD1.2
- net DS/CD1: no longer SD1.CD1
- net DTR: now also U3.1
- net GND: no longer C21.2, SD1.6, SD1.MT1, SD1.MT2, U4.4
- net MISO: no longer SD1.7
- net MOSI: no longer SD1.3
- net N$4: now also Y1.P$1; no longer XTAL1.P$1
- net N$6: now also Y1.P$2; no longer XTAL1.P$2
- net SCK: no longer SD1.5
- net SCL: no longer U4.6
- net SDA: no longer U4.5
- net VIN: no longer C1.2, C3.2, CHRG1.4, LDO1.1, LDO1.3, R3.2
Routing:
- net DTR: track 0.00 -> 36.2 mm, vias 0 -> 2
- net RXD.NRF: track 0.00 -> 30.4 mm, vias 0 -> 2
- net GND: track 28.3 -> 56.2 mm, vias 19 -> 29
- net RESET: track 0.00 -> 26.8 mm, vias 0 -> 1
- net D15/SW2: track 0.00 -> 23.9 mm, vias 0 -> 2
- net TXD.NRF: track 0.00 -> 23.9 mm, vias 0 -> 2
- net SCL: track 0.00 -> 23.7 mm, vias 0 -> 1
- net A7/BATT: track 0.00 -> 22.4 mm, vias 0 -> 2
- net RXD.FT: track 0.00 -> 20.8 mm
- net SDA: track 0.00 -> 20.4 mm, vias 0 -> 1
- net D11/SW1: track 0.00 -> 19.4 mm
- net D16/CS.OLED: track 0.00 -> 18.6 mm, vias 0 -> 2
- net VIN1: track 0.00 -> 17.1 mm, vias 0 -> 1
- net SCK: track 0.00 -> 17.1 mm, vias 0 -> 2
- net MOSI: track 0.00 -> 15.7 mm, vias 0 -> 2
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
Commit message: Take 7 Finished;
Parts:
- moved LDO1 43.5 mm to (9.98, 26.9), turned to 270 degrees
- moved C6 42.3 mm to (9.67, 29.4), turned to 180 degrees
- moved C3 3.87 mm to (4.84, 27.0), turned to 90 degrees
- moved C1 2.52 mm to (7.28, 27.1)
- moved R4 1.50 mm to (2.45, 29.6), turned to 180 degrees
- moved R3 0.97 mm to (5.78, 29.6), turned to 0 degrees
- moved R6 0.34 mm to (2.43, 19.4)
- moved Y1 0.20 mm to (18.4, 21.5)
Connections:
- removed net VIN1: C1.2, C3.2, CHRG1.4, LDO1.1, LDO1.3, R3.2
- net VIN: now also C1.2, C3.2, CHRG1.4, LDO1.1, LDO1.3, R3.2
Routing:
- net VIN: track 1.56 -> 41.3 mm, vias 0 -> 1
- net D27/CHRG.STATUS: track 0.00 -> 28.2 mm, vias 0 -> 5
- net VIN1: track 17.1 -> 0.00 mm, vias 1 -> 0
- net GND: track 56.2 -> 65.0 mm, vias 29 -> 30
- net RXD.FT: track 20.8 -> 16.5 mm
- net N$17: track 0.00 -> 1.50 mm
- net N$11: track 8.76 -> 7.76 mm
- net A4/PPG: track 10.2 -> 11.2 mm
- net N$3: track 4.99 -> 4.06 mm
- net VLIPO: track 29.8 -> 30.4 mm
- net SCL: track 23.7 -> 23.1 mm
- net A7/BATT: track 22.4 -> 23.0 mm

Commit message: Take 7 Done w/ no airwire
Routing:
- net N$4: track 8.03 -> 7.44 mm
Changed lines of the file:
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@@
 <contactref element="Y1" pad="P$1"/>
 <contactref element="U1" pad="13"/>
-<wire x1="18.060278125" y1="20.812853125" x2="17.89208125" y2="20.64465625" width="0.1524" layer="1"/>
 <wire x1="15.392403125" y1="21.362296875" x2="15.392403125" y2="21.204815625" width="0.1524" layer="1"/>
-<wire x1="18.279821875" y1="20.52019375" x2="18.44801875" y2="20.688390625" width="0.1524" layer="1"/>
-<wire x1="18.44801875" y1="20.688390625" x2="18.43381875" y2="20.674190625" width="0.2" layer="1"/>
-<wire x1="18.43381875" y1="20.674190625" x2="15.923028125" y2="20.674190625" width="0.2" layer="1"/>
-<wire x1="15.392403125" y1="21.204815625" x2="15.923028125" y2="20.674190625" width="0.2" layer="1"/>
-<wire x1="18.44801875" y1="20.688390625" x2="21.259890625" y2="20.688390625" width="0.2" layer="1"/>
-<wire x1="21.259890625" y1="20.688390625" x2="21.48078125" y2="20.90928125" width="0.2" layer="1"/>
-<wire x1="21.48078125" y1="20.90928125" x2="21.48078125" y2="21.872540625" width="0.2" layer="1"/>
 <wire x1="21.48078125" y1="21.872540625" x2="21.45804375" y2="21.895278125" width="0.2" layer="1"/>
-<wire x1="18.279821875" y1="20.52019375" x2="18.060278125" y2="20.812853125" width="0" layer="19" extent="1-1"/>
+<wire x1="15.392403125" y1="21.362296875" x2="16.080509375" y2="20.674190625" width="0.2" layer="1"/>
+<wire x1="16.080509375" y1="20.674190625" x2="17.467603125" y2="20.674190625" width="0.2" layer="1"/>
+<wire x1="21.250440625" y1="20.990728125" x2="21.250440625" y2="21.6422" width="0.2" layer="1"/>
+<wire x1="21.250440625" y1="21.6422" x2="21.48078125" y2="21.872540625" width="0.2" layer="1"/>
+<wire x1="20.948103125" y1="20.688390625" x2="21.250440625" y2="20.990728125" width="0.2" layer="1"/>
+<wire x1="17.467603125" y1="20.674190625" x2="17.481803125" y2="20.688390625" width="0.2" layer="1"/>
+<wire x1="17.481803125" y1="20.688390625" x2="18.44801875" y2="20.688390625" width="0.2" layer="1"/>
+<wire x1="18.44801875" y1="20.688390625" x2="20.948103125" y2="20.688390625" width="0.2" layer="1"/>
 </signal>
 <signal name="N$6">

Commit message: Finished take 8!
Parts:
- renumbered SW1 to RESET, SW2 to DFU
Other:
- board text added: "+"
