File: Hardware/Top/cataclysm-TOP.sch (EAGLE design)
At the start: 0 parts

Commit message: Added OLED display, power management section, bluetooth microcontroller, and buttons
Parts:
- added C10, C11: 300p, LinnesLab-Passives:CAPACITOR0603
- added C12: 10u, LinnesLab-Passives:CAPACITOR0805
- added C13, C15, C17, C18, C19: 2.2uF, LinnesLab-Passives:CAPACITOR0402
- added C14: 100n, LinnesLab-Passives:CAPACITOR0603
- added C16: 10uF, LinnesLab-Passives:CAPACITOR0603
- added C2, C5, C6, C7: 1u, LinnesLab-Passives:CAPACITOR0603
- added C20, C21: 4.7u, LinnesLab-Passives:CAPACITOR0603
- added C8, C9: (no value), LinnesLab-Passives:CAPACITOR0603
- added CHRG2: MCP73831, LinnesLab-Power:MCP73831
- added CORTEX1: CORTEX_DEBUG_PTH, LinnesLab-Connectors:CORTEX_DEBUG_PTH
- added D1, D4, D5: (no value), LinnesLab-DiscreteSemi:SCHOTTKY-USC
- added J2: (no value), LinnesLab-Connectors:CONN_02
- added L2: 10u, LinnesLab-Passives:INDUCTOR0603
- added LDO2: MIC5504, LinnesLab-Power:MIC5504
- added LED3: RED, LinnesLab-LED:LED0603
- added LED4: BLUE, LinnesLab-LED:LED0603
- added R11: (no value), LinnesLab-Passives:RESISTOR0603
- added R12, R13, R14, R15: 100k, LinnesLab-Passives:RESISTOR0603
- added R3, R4: 1k, LinnesLab-Passives:RESISTOR0603
- added R5, R6, R8, R9: 10k, LinnesLab-Passives:RESISTOR0603
- added R7: 390k, LinnesLab-Passives:RESISTOR0603
- added SD3: (no value), LinnesLab-Connectors:MICROSD
- added SW1, SW2, SW5: SWITCH.MOM, LinnesLab-Switches:SWITCH.MOM
- added SW3, SW4: (no value), LinnesLab-Switches:SPST-PTS830GG140-COPY.1-3
- added U2: NRF52832_MODULE_MDBT42, LinnesLab-Microcontrollers:NRF52832_MODULE_MDBT42
- added U3: (no value), LinnesLab-Displays:DISP_OLED_UG-2864HSWEG01-NO-WRAPAROUND
- added U4: PCF8523, LinnesLab-Clocks:PCF8523
- added USB2: USB.MICRO-BIGGERPADS, LinnesLab-Connectors:USB.MICRO-BIGGERPADS
- added XTAL2: 32.768kHz, LinnesLab-Clocks:CRYSTALECS-.327-12.5-12-C-TR
- added XTAL3: 32.7680kHz, LinnesLab-Clocks:CRYSTALECS-.327-12.5-12-C-TR
Connections:
- new net 3.3V: C12.2, C17.2, C19.2, C2.1, C6.1, CORTEX1.VCC, D1.C, LDO2.OUT, R15.2, R5.2, R8.2, R9.2, SD3.VDD, U2.VDD, U3.VBAT, U3.VDD, U4.VDD
- new net BATT: R13.1, R14.2
- new net CD1: SD3.CARD_DETECT
- new net CD2: SD3.CARD_DETECT1
- new net CHRG.STAT: CHRG2.STAT, R12.1
- new net CS.OLED: U3./CS
- new net DC.OLED: U3.DC/I2C_SA0
- new net DFU: SW3.B, U2.P0.20
- new net DTR: C14.1
- new net FRST: U2.P0.22
- new net GND: C10.2, C11.2, C12.1, C16.1, C17.1, C18.1, C19.1, C2.2, C20.2, C21.1, C5.1, C6.2, C7.2, C8.1, C9.2, CHRG2.VSS, CORTEX1.GND@3, CORTEX1.GND@5, CORTEX1.GNDDTCT, CORTEX1.KEY, J2.1, LDO2.GND, LED3.C, LED4.C, R11.1, R14.1, R15.1, R6.1, R7.2, SD3.GND, SD3.GND1, SD3.VSS, SW3.A, SW4.B, U2.GND@1, U2.GND@2, U2.GND@3, U2.GND@4, U3.BS0, U3.BS2, U3.NC(GND)@1, U3.NC(GND)@2, U3.VLSS, U3.VSS, U4.VSS, USB2.GND
- new net LED1: R3.2, U2.P0.17
- new net LED2: R4.2, U2.P0.19
- new net MISO: SD3.DATA_OUT, U2.P0.14
- new net MOSI: SD3.DATA_IN, U2.P0.13, U3.D1/SPI_SDIN/I2C_SDA
- new net N$1: R6.2, U3.BS1
- new net N$10: LED4.A, R4.1
- new net N$11: L2.1, U2.DCC
- new net N$12: C7.1, L2.2, U2.DEC4
- new net N$13: C16.2, U3.VCC
- new net N$14: CORTEX1.NC/TDI
- new net N$15: C18.2, U3.VCOMH
- new net N$17: CHRG2.PROG, R11.2
- new net N$19: U4.OSCO, XTAL3.1
- new net N$2: R7.1, U3.IREF
- new net N$20: U4.OSCI, XTAL3.2
- new net N$3: C13.2, U3.C2P
- new net N$4: C8.2, U2.P0.00/XL1, XTAL2.1
- new net N$5: C13.1, U3.C2N
- new net N$6: C9.1, U2.P0.01/XL2, XTAL2.2
- new net N$7: C15.2, U3.C1P
- new net N$8: C15.1, U3.C1N
- new net N$9: LED3.A, R3.1
- new net P0.09/NFC1: C11.1, U2.P0.09
- new net P0.10/NFC2: C10.1, U2.P0.10
- new net RESET: C14.2, CORTEX1.!RESET, D1.A, R5.1, SW4.A, U2.P0.21/RESET
- new net RESET.OLED: U3./RES
- new net RXD: U2.P0.08
- new net SCK: SD3.SCLK, U2.P0.12, U3.D0/SPI_SCLK/I2C_SCK
- new net SCL: R8.1, U2.P0.26, U4.SCL
- new net SD.CS: SD3.CS
- new net SDA: R9.1, U2.P0.25, U4.SDA
- new net SWCLK: CORTEX1.SWDCLK/TCK, U2.SWDCLK
- new net SWDIO: CORTEX1.SWDIO/TMS, U2.SWDIO
- new net SWO: CORTEX1.SWO/TDO, U2.P0.18/SWO
- new net TXD: U2.P0.06
- new net USB+: USB2.D+
- new net USB-: USB2.D-
- new net VBATT: U4.VBAT
- new net VIN: C21.2, C5.2, CHRG2.VIN, D4.C, D5.C, LDO2.EN, LDO2.IN, R12.2
- new net VLIPO: C20.1, CHRG2.VBAT, D4.A, J2.2, R13.2
- new net V_USB: D5.A, USB2.V+
Other:
- note added: "100nF+10K @ 3.3V = ~1.2ms to 0.7VCC"
- note added: "Additional notes for advanced users only"
- note added: "Back-up battery if desired"
- note added: "Connect MISO, MOSI, and SCK to appropriate pins on microcontroller. Those are SPI pins and are generally prespecified. You have more flexibility with the SD.CS pin."
- note added: "I2C Address = 0x68h"
- note added: "Microcontroller Reset Circuit"
- note added: "OLED"
- note added: "PIN_DFU / P0.20: If this pin is detected to be at GND level at startup, the board will enter a special serial bootloader mode and will not execute any user code, going straight into bootloader mode. If you wish to use this pin as a standard GPIO, make sure that it is pulled high with a pullup resistor so that your code will execute normally when the MCU starts up. FRST/P0.22: Setting this pin to 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"
- note added: "SPECIAL / PORT / PIN ON PACKAGE / GPIO(D_or_A) / Comments Factory Reset / P0.22 / pin38 / DO NOT USE FOR ANY GPIO SWDIO / none / pin37 / reserved-not available for general GPIO SWCLK / none / pin36 / reserved-not available for general GPIO RESET / P0.21 / pin35 / reserved-not available for general GPIO DFU / P0.20 / pin34 / reserved-not available for general GPIO LED2 / P0.19 / pin33 / reserved f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"
- note added: "SPECIAL / PORT / PIN ON PACKAGE / GPIO(D_or_A) / Comments SDA / P0.25 / pin2 / D25 SCL / P0.26 / pin3 / D26 none / P0.27 / pin4 / D27 none / P0.28 / pin5 / D28_or_A4 / (low drive, low frequency IO) none / P0.29 / pin6 / D29_or_A5 / (low drive, low frequency IO) none / P0.30 / pin7 / D30_or_A6 none / P0.31 / pin8 / D31_or_A7 / (used for battery level monitoring on Adafruit boards)"
- note added: "SPECIAL / PORT / PIN ON PACKAGE / GPIO(D_or_A) / Comments none / P0.02 / pin15 / D2_or_A0 none / P0.03 / pin16 / D3_or_A1 none / P0.04 / pin17 / D4_or_A2 none / P0.05 / pin18 / D5_or_A3 TXD / P0.06 / pin19 / D6 / but reserved for Serial communication and programming none / P0.07 / pin20 / D7 RXD / P0.08 / pin21 / D8 / but reserved for Serial communication and programming NFC1 / P0.09 / pin22 / D9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"
- note added: "Some pins are noted as reserved and not available for general GPIO (unless you are an adavanced user) I2C, SPI, and SWD pins can be repurposed if you know what you are doing For Milestones, avoid repurposing NFC pins. For P0.19 (LED2), Adafruit's Bluetooth Low Energy libraries use this pin to indicated successful pairing. The LED blinks when the device is doing some Bluetooth process and stays li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"

Commit message: complete top circuit schematic
Parts:
- removed SW5: SWITCH.MOM, LinnesLab-Switches:SWITCH.MOM
Connections:
- new net N$16: SW2.4
- new net N$21: SW1.4
- new net SW1: SW1.1, SW2.1
- net GND: now also SW1.3, SW2.3, USB2.SHIELD
Other:
- note added: "Buttons"
- note added: "Cortex Debugger / Programmer"
- note added: "Digital GPIO CS.OLED RESET.OLED DC.OLED Digital Inputs 3x buttons Charge Status Analog Inputs Battery monitor Analog Output"
- note added: "Power Management"
- note added: "Real-Time Clock"
- note added: "SD Card"
- note added: "nRF52832 Module"
- moved on the sheet: C10, C11, C12, C13, C14, C15, C16, C17, C18, C19, C2, C20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

Commit message: Finished top and bottom schematic
Parts:
- added C22: 100n, LinnesLab-Passives:CAPACITOR0603
- added C23, C24: 47p, LinnesLab-Passives:CAPACITOR0603
- added J1: (no value), LinnesLab-Connectors:CONN_07-1.27MM
- added JP2: (no value), LinnesLab-Switches:JUMPER-SMT_2_NO_SILK
- added LED5: RED, LinnesLab-LED:LED0603
- added LED6: YELLOW, LinnesLab-LED:LED0603
- added R1, R2: 0, LinnesLab-Passives:RESISTOR0603
- added R17, R18: 27, LinnesLab-Passives:RESISTOR0603
- added R19, R20: 1k, LinnesLab-Passives:RESISTOR0603
- added U5: FT231XS, LinnesLab-DigitalIC:FT231XS
Connections:
- removed net BATT: R13.1, R14.2
- removed net CD1: SD3.CARD_DETECT
- removed net CHRG.STAT: CHRG2.STAT, R12.1
- removed net CS.OLED: U3./CS
- removed net DC.OLED: U3.DC/I2C_SA0
- removed net RESET.OLED: U3./RES
- removed net RXD: U2.P0.08
- removed net SD.CS: SD3.CS
- removed net SW1: SW1.1, SW2.1
- removed net TXD: U2.P0.06
- removed net VBATT: U4.VBAT
- new net !CTS: JP2.2, U5.!CTS
- new net !DTR: U5.!DTR
- new net A4/BATT: U2.P0.28/AIN4
- new net A6/TIA: U2.P0.30/AIN6
- new net A7/PPG: J1.7, U2.P0.31/AIN7
- new net A7/TIA: J1.5
- new net D11/SW1: SW1.1, U2.P0.11
- new net D15/SW2: SW2.1, U2.P0.15
- new net D16/CS.OLED: U2.P0.16, U3./CS
- new net D27/CHRG.STATUS: CHRG2.STAT, R12.1, R13.1, R14.2, U2.P0.27
- new net D29/LED.CTRL: J1.6, U2.P0.29/AIN5
- new net D3/RESET.OLED: U2.P0.04/AIN2, U3./RES
- new net D4/DC.OLED: U2.P0.03/AIN1, U3.DC/I2C_SA0
- new net D7/SD.CS: SD3.CS, U2.P0.07
- new net DS/CD1: SD3.CARD_DETECT, U2.P0.05/AIN3
- new net FT3V3: U5.3V3OUT
- new net N$24: J1.4
- new net N$25: R17.2, U5.USBDM
- new net N$26: R18.2, U5.USBDP
- new net N$27: LED5.C, R19.2
- new net N$28: LED6.C, R20.2
- new net N$29: J1.3
- new net N$30: J1.2
- new net N$31: J1.1
- new net RXD.FT: R2.1, U5.RXD
- new net RXD.NRF: R1.2, U2.P0.08
- new net RXLED: R19.1, U5.CBUS1
- new net TXD.FT: R1.1, U5.TXD
- new net TXD.NRF: R2.2, U2.P0.06
- new net TXLED: R20.1, U5.CBUS2
- net 3.3V: now also C22.2, LED5.A, LED6.A, U5.!RESET, U5.VCCIO
- net GND: now also C22.1, C23.2, C24.1, JP2.1, U5.GND@16, U5.GND@6
- net SCL: now also R9.1; no longer R8.1
- net SDA: now also R8.1; no longer R9.1
- net USB+: now also C23.1, R18.1
- net USB-: now also C24.2, R17.1
- net V_USB: now also U5.VCC
Other:
- note added: "Digital Output"
- note added: "FTDI Serial-to-USB Convertor"
- note added: "I don't remember if CTS needs to be grounded or left floating so here's a jumper to ground so it can be configued either way dynamically."
- note added: "Notes"
- note added: "TXD goes to RX on the other device RXD goes to TX on the other device"
- note removed: "Back-up battery if desired"
- moved on the sheet: C10, C11, C12, C13, C14, C15, C16, C17, C18, C19, C2, C20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

Commit message: Updated top board
Parts:
- removed C10: 300p, LinnesLab-Passives:CAPACITOR0603
- removed C22: 100n, LinnesLab-Passives:CAPACITOR0603
- removed C23, C24: 47p, LinnesLab-Passives:CAPACITOR0603
- removed C9: (no value), LinnesLab-Passives:CAPACITOR0603
- removed D4: (no value), LinnesLab-DiscreteSemi:SCHOTTKY-USC
- removed LED5: RED, LinnesLab-LED:LED0603
- removed LED6: YELLOW, LinnesLab-LED:LED0603
- removed R19: 1k, LinnesLab-Passives:RESISTOR0603
- removed R5: 10k, LinnesLab-Passives:RESISTOR0603
- removed U5: FT231XS, LinnesLab-DigitalIC:FT231XS
- removed XTAL3: 32.7680kHz, LinnesLab-Clocks:CRYSTALECS-.327-12.5-12-C-TR
- added C1: 4.7u, LinnesLab-Passives:CAPACITOR0603
- added C3: 1u, LinnesLab-Passives:CAPACITOR0603
- added C4: 10u, LinnesLab-Passives:CAPACITOR0805
- added D3: (no value), LinnesLab-DiscreteSemi:SCHOTTKY-USC
- added LED1: RED, LinnesLab-LED:LED0603
- added LED2: BLUE, LinnesLab-LED:LED0603
- added R10: 1k, LinnesLab-Passives:RESISTOR0603
- added U1: NRF52832_MODULE_MDBT42, LinnesLab-Microcontrollers:NRF52832_MODULE_MDBT42
- added XTAL1: 32.768kHz, LinnesLab-Clocks:CRYSTALECS-.327-12.5-12-C-TR
- C11: value 300p -> 100n
- C12: value 10u -> 10uF; device LinnesLab-Passives:CAPACITOR0805 -> LinnesLab-Passives:CAPACITOR0603
- C14: value 100n -> 2.2uF; device LinnesLab-Passives:CAPACITOR0603 -> LinnesLab-Passives:CAPACITOR0402
- C16: value 10uF -> 2.2uF; device LinnesLab-Passives:CAPACITOR0603 -> LinnesLab-Passives:CAPACITOR0402
- C18, C19: value 2.2uF -> 47p; device LinnesLab-Passives:CAPACITOR0402 -> LinnesLab-Passives:CAPACITOR0603
- C20: value 4.7u -> 100n
- C21: value 4.7u -> 1u
- C5, C7: value 1u -> (none)
- C8: value (none) -> 4.7u
- J1: device LinnesLab-Connectors:CONN_07-1.27MM -> LinnesLab-Connectors:CONN_02
- J2: device LinnesLab-Connectors:CONN_02 -> LinnesLab-Connectors:CONN_07-1.27MM
- LED4: value BLUE -> YELLOW
- R1, R2: value 0 -> 10k
- R11: value (none) -> 10k
- R12: value 100k -> 390k
- R13, R14: value 100k -> 27
- R15: value 100k -> 1k
- R17, R18: value 27 -> 0
- R3: value 1k -> 100k
- R4: value 1k -> (none)
- R6: value 10k -> 100k
- R7: value 390k -> 100k
- R9: value 10k -> 1k
- SW1, SW2: value SWITCH.MOM -> (none); device LinnesLab-Switches:SWITCH.MOM -> LinnesLab-Switches:SPST-PTS830GG140-COPY.1-3
- SW3, SW4: value (none) -> SWITCH.MOM; device LinnesLab-Switches:SPST-PTS830GG140-COPY.1-3 -> LinnesLab-Switches:SWITCH.MOM
- U2: value NRF52832_MODULE_MDBT42 -> (none); device LinnesLab-Microcontrollers:NRF52832_MODULE_MDBT42 -> LinnesLab-Displays:DISP_OLED_UG-2864HSWEG01-NO-WRAPAROUND
- U3: value (none) -> FT231XS; device LinnesLab-Displays:DISP_OLED_UG-2864HSWEG01-NO-WRAPAROUND -> LinnesLab-DigitalIC:FT231XS
- XTAL2: value 32.768kHz -> 32.7680kHz; FREQ (none) -> 32.7680KHZ
- renumbered CHRG2 to CHRG1, CORTEX1 to DEBUG1, D5 to D2, JP2 to JP1, L2 to L1, LDO2 to LDO1, R20 to R16, SD3 to SD1, USB2 to USB1
Connections:
- removed net A7/TIA: J1.5
- removed net N$24: J1.4
- removed net N$29: J1.3
- removed net N$30: J1.2
- removed net N$31: J1.1
- net !CTS: now also U3.!CTS; no longer U5.!CTS
- net !DTR: now also U3.!DTR; no longer U5.!DTR
- net 3.3V: now also C16.2, C20.2, C21.1, C4.2, D3.C, J2.4, LED3.A, LED4.A, R1.2, R2.2, U1.VDD, U2.VBAT, U3.!RESET, U3.VCCIO; no longer C12.2, C19.2, C2.1, C22.2, D1.C, LED5.A, LED6.A, R15.2, R5.2, R9.2, U3.VBAT, U3.VDD, U5.!RESET, U5.VCCIO
- net A4/BATT: now also R6.1, R7.2, U1.P0.28/AIN4; no longer U2.P0.28/AIN4
- net A6/TIA: now also J2.6, U1.P0.30/AIN6; no longer U2.P0.30/AIN6
- net A7/PPG: now also J2.7, U1.P0.31/AIN7; no longer J1.7, U2.P0.31/AIN7
- net D11/SW1: now also SW3.1, U1.P0.11; no longer SW1.1, U2.P0.11
- net D15/SW2: now also SW4.1, U1.P0.15; no longer SW2.1, U2.P0.15
- net D16/CS.OLED: now also U1.P0.16, U2./CS; no longer U2.P0.16, U3./CS
- net D27/CHRG.STATUS: now also R3.1, U1.P0.27; no longer R12.1, R13.1, R14.2, U2.P0.27
- net D29/LED.CTRL: now also J2.5, U1.P0.29/AIN5; no longer J1.6, U2.P0.29/AIN5
- net D3/RESET.OLED: now also U1.P0.04/AIN2, U2./RES; no longer U2.P0.04/AIN2, U3./RES
- net D4/DC.OLED: now also U1.P0.03/AIN1, U2.DC/I2C_SA0; no longer U2.P0.03/AIN1, U3.DC/I2C_SA0
- net D7/SD.CS: now also U1.P0.07; no longer U2.P0.07
- net DFU: now also SW2.B, U1.P0.20; no longer SW3.B, U2.P0.20
- net DS/CD1: now also U1.P0.05/AIN3; no longer U2.P0.05/AIN3
- net DTR: now also C11.1; no longer C14.1
- net FRST: now also U1.P0.22; no longer U2.P0.22
- net FT3V3: now also U3.3V3OUT; no longer U5.3V3OUT
- net GND: now also C1.1, C14.1, C19.2, C20.1, C21.2, C3.1, C4.1, C8.2, J1.1, J2.3, LED1.C, LED2.C, R12.2, R4.1, R7.1, SW1.B, SW2.A, SW3.3, SW4.3, U1.GND@1, U1.GND@2, U1.GND@3, U1.GND@4, U2.BS0, U2.BS2, U2.NC(GND)@1, U2.NC(GND)@2, U2.VLSS, U2.VSS, U3.GND@16, U3.GND@6; no longer C10.2, C11.2, C19.1, C20.2, C21.1, C22.1, C23.2, C24.1, C8.1, C9.2, J2.1, LED3.C, LED4.C, R14.1, R15.1, R6.1, R7.2, SW1.3, SW2.3, SW3.A, SW4.B, U2.GND@1, U2.GND@2, U2.GND@3, U2.GND@4, U3.BS0, U3.BS2, U3.NC(GND)@1, U3.NC(GND)@2, U3.VLSS, U3.VSS, U5.GND@16, U5.GND@6
- net LED1: now also R9.2, U1.P0.17; no longer R3.2, U2.P0.17
- net LED2: now also R10.2, U1.P0.19; no longer R4.2, U2.P0.19
- net MISO: now also U1.P0.14; no longer U2.P0.14
- net MOSI: now also U1.P0.13, U2.D1/SPI_SDIN/I2C_SDA; no longer U2.P0.13, U3.D1/SPI_SDIN/I2C_SDA
- net N$1: now also R11.2, U2.BS1; no longer R6.2, U3.BS1
- net N$10: now also LED2.A, R10.1; no longer LED4.A, R4.1
- net N$11: now also U1.DCC; no longer U2.DCC
- net N$12: now also C2.1, U1.DEC4; no longer C7.1, U2.DEC4
- net N$13: now also C12.2, U2.VCC; no longer C16.2, U3.VCC
- net N$15: now also C14.2, U2.VCOMH; no longer C18.2, U3.VCOMH
- net N$16: now also SW4.4; no longer SW2.4
- net N$17: now also R4.2; no longer R11.2
- net N$19: now also XTAL2.1; no longer XTAL3.1
- net N$2: now also R12.1, U2.IREF; no longer R7.1, U3.IREF
- net N$20: now also XTAL2.2; no longer XTAL3.2
- net N$21: now also SW3.4; no longer SW1.4
- net N$25: now also R13.2, U3.USBDM; no longer R17.2, U5.USBDM
- net N$26: now also R14.2, U3.USBDP; no longer R18.2, U5.USBDP
- net N$27: now also LED3.C, R15.2; no longer LED5.C, R19.2
- net N$28: now also LED4.C; no longer LED6.C
- net N$3: now also C15.2, U2.C2P; no longer C13.2, U3.C2P
- net N$4: now also C5.2, U1.P0.00/XL1, XTAL1.1; no longer C8.2, U2.P0.00/XL1, XTAL2.1
- net N$5: now also C15.1, U2.C2N; no longer C13.1, U3.C2N
- net N$6: now also C7.1, U1.P0.01/XL2, XTAL1.2; no longer C9.1, U2.P0.01/XL2, XTAL2.2
- net N$7: now also C13.2, U2.C1P; no longer C15.2, U3.C1P
- net N$8: now also C13.1, U2.C1N; no longer C15.1, U3.C1N
- net N$9: now also LED1.A, R9.1; no longer LED3.A, R3.1
- net P0.09/NFC1: now also U1.P0.09; no longer C11.1, U2.P0.09
- net P0.10/NFC2: now also U1.P0.10; no longer C10.1, U2.P0.10
- net RESET: now also C11.2, D3.A, R8.1, SW1.A, U1.P0.21/RESET; no longer C14.2, D1.A, R5.1, SW4.A, U2.P0.21/RESET
- net RXD.FT: now also R18.1, U3.RXD; no longer R2.1, U5.RXD
- net RXD.NRF: now also R17.2, U1.P0.08; no longer R1.2, U2.P0.08
- net RXLED: now also R15.1, U3.CBUS1; no longer R19.1, U5.CBUS1
- net SCK: now also U1.P0.12, U2.D0/SPI_SCLK/I2C_SCK; no longer U2.P0.12, U3.D0/SPI_SCLK/I2C_SCK
- net SCL: now also J2.2, R2.1, U1.P0.26; no longer R9.1, U2.P0.26
- net SDA: now also J2.1, R1.1, U1.P0.25; no longer R8.1, U2.P0.25
- net SWCLK: now also U1.SWDCLK; no longer U2.SWDCLK
- net SWDIO: now also U1.SWDIO; no longer U2.SWDIO
- net SWO: now also U1.P0.18/SWO; no longer U2.P0.18/SWO
- net TXD.FT: now also R17.1, U3.TXD; no longer R1.1, U5.TXD
- net TXD.NRF: now also R18.2, U1.P0.06; no longer R2.2, U2.P0.06
- net TXLED: now also U3.CBUS2; no longer U5.CBUS2
- net USB+: now also C19.1, R14.1; no longer C23.1, R18.1
- net USB-: now also C18.2, R13.1; no longer C24.2, R17.1
- net VIN: now also C1.2, C3.2, D1.C, R3.2; no longer C21.2, C5.2, D4.C, R12.2
- net VLIPO: now also C8.1, D1.A, J1.2, R6.2; no longer C20.1, D4.A, J2.2, R13.2
- net V_USB: now also U3.VCC; no longer U5.VCC
Other:
- note added: "Connection to Bottom Board"
- moved on the sheet: C11, C12, C13, C14, C15, C16, C18, C19, C2, C20, C21, C5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

Commit message: Almost finished with take 8
Parts:
- removed C21: 1u, LinnesLab-Passives:CAPACITOR0603
- removed SD1: (no value), LinnesLab-Connectors:MICROSD
- removed U4: PCF8523, LinnesLab-Clocks:PCF8523
- removed XTAL2: 32.7680kHz, LinnesLab-Clocks:CRYSTALECS-.327-12.5-12-C-TR
- C1: value 4.7u -> 1u
- C14: device LinnesLab-Passives:CAPACITOR0402 -> LinnesLab-Passives:CAPACITOR0603
- C3: value 1u -> 4.7u
- renumbered XTAL1 to Y1
Connections:
- removed net !DTR: U3.!DTR
- removed net A4/BATT: R6.1, R7.2, U1.P0.28/AIN4
- removed net A7/PPG: J2.7, U1.P0.31/AIN7
- removed net CD2: SD1.CARD_DETECT1
- removed net N$19: U4.OSCO, XTAL2.1
- removed net N$20: U4.OSCI, XTAL2.2
- new net A4/PPG: J2.7, U1.P0.28/AIN4
- new net A7/BATT: R6.1, R7.2, U1.P0.31/AIN7
- new net VIN1: C1.2, C3.2, CHRG1.VIN, LDO1.EN, LDO1.IN, R3.2
- net 3.3V: no longer C21.1, SD1.VDD, U4.VDD
- net A6/TIA: now also J2.5; no longer J2.6
- net D29/LED.CTRL: now also J2.6; no longer J2.5
- net D7/SD.CS: no longer SD1.CS
- net DS/CD1: no longer SD1.CARD_DETECT
- net DTR: now also U3.!DTR
- net GND: no longer C21.2, SD1.GND, SD1.GND1, SD1.VSS, U4.VSS
- net MISO: no longer SD1.DATA_OUT
- net MOSI: no longer SD1.DATA_IN
- net SCK: no longer SD1.SCLK
- net SCL: no longer U4.SCL
- net SDA: no longer U4.SDA
- net VIN: no longer C1.2, C3.2, CHRG1.VIN, LDO1.EN, LDO1.IN, R3.2
Other:
- note removed: "Connect MISO, MOSI, and SCK to appropriate pins on microcontroller. Those are SPI pins and are generally prespecified. You have more flexibility with the SD.CS pin."
- note removed: "I2C Address = 0x68h"
- note removed: "Real-Time Clock"
- note removed: "SD Card"
- moved on the sheet: C1, C3

Commit message: Take 7 Finished;
Connections:
- removed net VIN1: C1.2, C3.2, CHRG1.VIN, LDO1.EN, LDO1.IN, R3.2
- net VIN: now also C1.2, C3.2, CHRG1.VIN, LDO1.EN, LDO1.IN, R3.2

Commit message: Finished take 8!
Parts:
- renumbered SW1 to RESET, SW2 to DFU
Other:
- note added: "0 ohm resistors in cass TX/RX are mixed up"
- note added: "Diodes switch from LiPo power to USB when USB is connected The USB then charges the battery"
- note added: "Headers connecting top and bottom board"
- note added: "R4 sets the charge current I_charge = 1000 V / R4 per MCP73831 datasheet"
- note added: "Voltage divider used to monitor battery voltage"
- note added: "cataclysm Basic Top July 2, 2020 Rev. 1 Purdue Milestones — Smartwatch Taught by Orlando Hoilett T.A. - Jason Uhmel - Nick Bluhm"
- note removed: "Connection to Bottom Board"
- moved on the sheet: C1, C3, C6, C8, CHRG1, D1, D2, J1, LDO1, R3, R4, R6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
